Commit message: Change origin rpy angles of joints 3 and 4

File: open_manipulator_p/open_manipulator_p_description/urdf/open_manipulator_p.urdf.xacro (robot description, xacro)
@@ -61,5 +61,5 @@
     <origin xyz="0.0 0.069 0.033" rpy="0 0 0"/>
     <axis xyz="0 1 0"/>
-    <limit velocity="6.5" effort="1000" lower="${-pi*0.5}" upper="${pi*0.5}" />
+    <limit velocity="6.5" effort="1000" lower="${-pi*0.452}" upper="${pi*0.472}" />
     <dynamics damping="0.7"/>
   </joint>
@@ -91,5 +91,5 @@
     <parent link="link3"/>
     <child link="link4"/>
-    <origin xyz="0.03000 -0.01150 0.26400" rpy="0 0 0"/>
+    <origin xyz="0.03000 -0.01150 0.26400" rpy="0 ${-pi * 44   / 180} 0"/>
     <axis xyz="0 1 0"/>
     <limit velocity="6.5" effort="1000" lower="${-pi*0.5}" upper="${pi*0.5}" />
@@ -123,5 +123,5 @@
     <parent link="link4"/>
     <child link="link5"/>
-    <origin xyz="0.19500 -0.05750 0.03000" rpy="0 0 0"/>
+    <origin xyz="0.19500 -0.05750 0.03000" rpy="${-pi / 2} 0 0"/>
     <axis xyz="1 0 0"/>
     <limit velocity="6.5" effort="1000" lower="${-pi*0.5}" upper="${pi*0.5}" />

Commit message: update urdf angular limits

File: open_manipulator_p/open_manipulator_p_description/urdf/open_manipulator_p.urdf.xacro (robot description, xacro)
@@ -61,5 +61,5 @@
     <origin xyz="0.0 0.069 0.033" rpy="0 0 0"/>
     <axis xyz="0 1 0"/>
-    <limit velocity="6.5" effort="1000" lower="${-pi*0.452}" upper="${pi*0.472}" />
+    <limit velocity="6.5" effort="1000" lower="${-pi*0.454}" upper="${pi*0.476}" />
     <dynamics damping="0.7"/>
   </joint>
@@ -93,5 +93,5 @@
     <origin xyz="0.03000 -0.01150 0.26400" rpy="0 ${-pi * 44   / 180} 0"/>
     <axis xyz="0 1 0"/>
-    <limit velocity="6.5" effort="1000" lower="${-pi*0.5}" upper="${pi*0.5}" />
+    <limit velocity="6.5" effort="1000" lower="${-pi*0.414}" upper="${pi*0.723}" />
     <dynamics damping="0.7"/>
   </joint>
@@ -125,5 +125,5 @@
     <origin xyz="0.19500 -0.05750 0.03000" rpy="${-pi / 2} 0 0"/>
     <axis xyz="1 0 0"/>
-    <limit velocity="6.5" effort="1000" lower="${-pi*0.5}" upper="${pi*0.5}" />
+    <limit velocity="6.5" effort="1000" lower="${-pi*0.494}" upper="${pi*0.494}" />
     <dynamics damping="0.7"/>
   </joint>
@@ -157,5 +157,5 @@
     <origin xyz="0.06300 0.04500 0.00000" rpy="0 0 0"/>
     <axis xyz="0 1 0"/>
-    <limit velocity="6.5" effort="1000" lower="${-pi*0.5}" upper="${pi*0.5}" />
+    <limit velocity="6.5" effort="1000" lower="${-pi*0.390}" upper="${pi*0.390}" />
     <dynamics damping="0.7"/>
   </joint>
@@ -189,5 +189,5 @@
     <origin xyz="0.12300 -0.04500 0.00000" rpy="0 0 0"/>
     <axis xyz="1 0 0"/>
-    <limit velocity="6.5" effort="1000" lower="${-pi*0.5}" upper="${pi*0.5}" />
+    <limit velocity="6.5" effort="1000" lower="${-pi}" upper="${pi}" />
     <dynamics damping="0.7"/>
   </joint>
