Commit message: add move_to.py script

File: open_manipulator_p/open_manipulator_p_description/urdf/camera.xacro (robot description, xacro)
@@ -7,5 +7,6 @@
         <parent link="link1"/>
         <child link="camera_link"/>
-        <origin xyz="0 0.07 0.04" rpy="0 ${-pi/6} 0"/>
+        <!-- <origin xyz="0 0.07 0.04" rpy="0 ${-pi/6} 0"/> -->
+        <origin xyz="0 0.07 0.04" rpy="0 ${-pi/18} 0"/>
     </joint>
     <link name="camera_link">

Commit message: fix aruco's tf offset error

File: open_manipulator_p/open_manipulator_p_description/urdf/camera.xacro (robot description, xacro)
@@ -8,5 +8,7 @@
         <child link="camera_link"/>
         <!-- <origin xyz="0 0.07 0.04" rpy="0 ${-pi/6} 0"/> -->
-        <origin xyz="0 0.07 0.04" rpy="0 ${-pi/18} 0"/>
+        <!-- <origin xyz="0 0.07 0.04" rpy="0 ${-pi/18} 0"/> -->
+        <origin xyz="0 0.14 0.14" rpy="0 0 0"/>
+        <!-- <origin xyz="0 1 1" rpy="0 0 0"/> -->
     </joint>
     <link name="camera_link">
@@ -40,5 +42,5 @@
             <update_rate>10</update_rate>
             <camera>
-                <horizontal_fov>1.3962634</horizontal_fov>
+                <horizontal_fov>1.089</horizontal_fov>
                 <image>
                     <format>R8G8B8</format>

Commit message: change camera urdf position

File: open_manipulator_p/open_manipulator_p_description/urdf/camera.xacro (robot description, xacro)
@@ -9,5 +9,5 @@
         <!-- <origin xyz="0 0.07 0.04" rpy="0 ${-pi/6} 0"/> -->
         <!-- <origin xyz="0 0.07 0.04" rpy="0 ${-pi/18} 0"/> -->
-        <origin xyz="0 0.14 0.14" rpy="0 0 0"/>
+        <origin xyz="0 0.20 0.14" rpy="0 0 0"/>
         <!-- <origin xyz="0 1 1" rpy="0 0 0"/> -->
     </joint>
